File: Preamplifier.kicad_pcb (KiCad board)
At the start: 2 copper layers, 163 parts, among them J1 Conn_01x02_Female, J10 AudioJack2, J12 XLR3, J13 Conn_01x03, J14 Conn_01x03, J15 Conn_01x02, J16 Conn_01x02, J17 Conn_01x02, J2 AudioJack2, J3 AudioJack3_SwitchTR, J4 AudioJack2_SwitchT, J5 AudioJack2_SwitchT, J6 Conn_01x02_Male, J7 Conn_01x02_Male, J8 Conn_01x05_Female, J9 AudioJack3_SwitchTR, Q1 2N3904, Q2 2N3906, Q3 2N3904, Q4 2N3906, Q5 BC549, SW1 SW_DPST, SW2 SW_SPDT, SW3 GND LIFT, U1 OPA2134, U2 NE5532, U3 NE5532, U4 NE5532, U5 TL072, U6 NE5532, U7 NE5532, U8 NE5532, U9 NE5532

Commit message: Did more work on amplifier
Parts:
- added J11: Conn_01x05_Female, TerminalBlock_Phoenix:TerminalBlock_Phoenix_PT-1,5-5-3.5-H_1x05_P3.50mm_Horizontal, F.Cu at (378.4, -10.4)
- added T1: Transformer_1P_2S, Project-152-Bass-Guitar-Amp:TE 49008024RC62, F.Cu at (23.0, 37.0)
- J1: footprint TerminalBlock_Phoenix:TerminalBlock_Phoenix_MKDS-1,5-2_1x02_P5.00mm_Horizontal -> TerminalBlock_Dinkle:TerminalBlock_Dinkle_DT-55-B01X-02_P10.00mm
- J6, J7: footprint TerminalBlock_Phoenix:TerminalBlock_Phoenix_PT-1,5-2-3.5-H_1x02_P3.50mm_Horizontal -> TerminalBlock_Phoenix:TerminalBlock_Phoenix_PT-1,5-2-5.0-H_1x02_P5.00mm_Horizontal
- moved C1 268.0 mm to (394.3, 42.6)
- moved C10 268.0 mm to (385.9, 37.0)
- moved C11 268.0 mm to (371.8, 57.2)
- moved C12 268.0 mm to (386.6, 58.3)
- moved C13 268.0 mm to (320.9, 83.4)
- moved C14 268.0 mm to (360.5, 67.4)
- moved C15 268.0 mm to (389.4, 55.3)
- moved C16 268.0 mm to (394.2, 51.4)
- moved C17 268.0 mm to (396.6, 33.5)
- moved C18 268.0 mm to (328.5, 65.4)
- moved C19 268.0 mm to (328.5, 71.3)
- moved C2 268.0 mm to (340.9, 85.1)
- moved C20 268.0 mm to (326.9, 94.0)
- moved C21 268.0 mm to (391.6, 48.5)
- moved C22 268.0 mm to (366.3, 77.7)
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- renumbered SW_HIGH_GAIN1 to SW4
Connections:
- D8 pad 2: Net-(D8-Pad2) -> (no net)
- J6 pad 1: Net-(F2-Pad2) -> (no net)
- J6 pad 2: Net-(F3-Pad1) -> (no net)
- J7 pad 1: Net-(F3-Pad2) -> (no net)
- R29 pad 1: Tuner -> (no net)
- R30 pad 1: EFXsend -> (no net)
- RV2 pad 2: Net-(J9-PadT) -> (no net)
- RV2 pad 5: Net-(J9-PadR) -> (no net)
Routing:
- net (no net): vias 0 -> 1
Other:
- board outline added: 200 x 95 mm
- board text added: "+12V"
- board text added: "-12V"
- board text added: "AUX IN"
- board text added: "EFFECTS RETURN"
- board text added: "FrEq"
- board text added: "GAIN"
- board text added: "GAIN SW"
- board text added: "GND"
- board text added: "GUITAR IN"
- board text added: "TO EFFECTS"
- board text added: "TO EQ BOARD"
- board text added: "ToEq"
- board text added: "WIP"
