File: Preamp/Preamplifier.sch (KiCad schematic (older format))
At the start: 155 parts, among them J1 Conn_01x03_Male, J12 XLR3, J14 Conn_01x03, J15 Conn_01x02, J16 Conn_01x02, J17 Conn_01x02, J2 Conn_01x02_Male, J3 Conn_01x02_Male, J4 Conn_01x03_Male, J5 Conn_01x03_Male, J6 Conn_01x02_Male, J7 Conn_01x03, J8 Conn_01x05_Female, Q1 2N3904, Q2 2N3906, Q3 2N3904, Q4 2N3906, Q5 BC549, SW1 SW_DPST, SW2 SW_SPDT, SW3 GND LIFT, SW4 SW_SPST, SW5 SW_HPFQ, U1 OPA2134, U2 NE5532, U3 NE5532, U4 NE5532, U5 TL072, U6 NE5532, U7 NE5532, U8 NE5532, U9 NE5532

Commit message: More layout work
Parts:
- removed C1, C2: 1uF, Capacitor_THT:C_Rect_L7.2mm_W7.2mm_P5.00mm_FKS2_FKP2_MKS2_MKP2, symbol Device:C
- removed C10, C11, C17: 100uF 50V, Capacitor_THT:CP_Radial_D8.0mm_P3.50mm, symbol Device:CP
- removed C12, C13, C15, C16, C18, C19, C20, C21, C22, C23, C24, C25, C26, C27, C28, C30, C33, C36, C37: 0.1uF, Capacitor_SMD:C_0805_2012Metric_Pad1.15x1.40mm_HandSolder, symbol Device:C
- removed C14: 100uF 50V, Capacitor_THT:CP_Radial_D8.0mm_P2.50mm, symbol Device:CP
- removed C29: 0.1uF (AUDIO), Capacitor_THT:C_Rect_L7.2mm_W2.5mm_P5.00mm_FKS2_FKP2_MKS2_MKP2, symbol Device:C
- removed C3, C6, C7, C9: 120n, Capacitor_THT:C_Rect_L7.2mm_W3.5mm_P5.00mm_FKS2_FKP2_MKS2_MKP2, symbol Device:C
- removed C32, C34, C35: 15nF, Capacitor_THT:C_Rect_L7.2mm_W2.5mm_P5.00mm_FKS2_FKP2_MKS2_MKP2, symbol Device:C
- removed C4: 47uF 63V, Capacitor_THT:CP_Radial_D8.0mm_P5.00mm, symbol Device:CP
- removed C41, C42, C43, C44: 100uF 63V, Capacitor_THT:CP_Radial_D8.0mm_P3.50mm, symbol Device:CP
- removed C5: 10uF 50V, Capacitor_THT:CP_Radial_D6.3mm_P2.50mm, symbol Device:CP
- removed D10, D11, D2, D3, D4, D5, D6, D7: 1N4148, Diode_THT:D_DO-35_SOD27_P7.62mm_Horizontal, symbol Diode:1N4148
- removed D12: OVERLOAD, LED_THT:LED_D3.0mm, symbol Device:LED
- removed D13: POWER, LED_THT:LED_D3.0mm, symbol Device:LED
- removed D14, D15, D16, D17: 10V, Diode_THT:D_DO-41_SOD81_P7.62mm_Horizontal, symbol Device:D_Zener
- removed J1, J4, J5: Conn_01x03_Male, Connector_PinHeader_2.54mm:PinHeader_1x03_P2.54mm_Vertical, symbol Connector:Conn_01x03_Male
- removed J12: XLR3, Connector_PinHeader_2.54mm:PinHeader_1x03_P2.54mm_Vertical, symbol Connector:XLR3
- removed J14: Conn_01x03, Connector_PinHeader_2.54mm:PinHeader_1x03_P2.54mm_Vertical, symbol Connector_Generic:Conn_01x03
- removed J15, J16, J17: Conn_01x02, Connector_PinHeader_2.54mm:PinHeader_1x02_P2.54mm_Vertical, symbol Connector_Generic:Conn_01x02
- removed J2, J3, J6: Conn_01x02_Male, Connector_PinHeader_2.54mm:PinHeader_1x02_P2.54mm_Vertical, symbol Connector:Conn_01x02_Male
- removed J7: Conn_01x03, TerminalBlock_Phoenix:TerminalBlock_Phoenix_MKDS-1,5-3_1x03_P5.00mm_Horizontal, symbol Connector_Generic:Conn_01x03
- removed J8: Conn_01x05_Female, Connector_PinHeader_2.54mm:PinHeader_1x05_P2.54mm_Vertical, symbol Connector:Conn_01x05_Female
- removed Q1, Q3: 2N3904, Package_TO_SOT_THT:TO-92_Inline, symbol Transistor_BJT:2N3904
- removed Q2, Q4: 2N3906, Package_TO_SOT_THT:TO-92_Inline, symbol Transistor_BJT:2N3906
- removed Q5: BC549, Package_TO_SOT_THT:TO-92_Inline, symbol Transistor_BJT:BC549
- removed R1, R39: 1M, Resistor_SMD:R_0805_2012Metric_Pad1.15x1.40mm_HandSolder, symbol Device:R
- removed R10, R11, R20, R22, R3, R31, R32, R48, R5, R52, R6, R8, R9: 10k, Resistor_SMD:R_0805_2012Metric_Pad1.15x1.40mm_HandSolder, symbol Device:R
- removed R12, R64: 33k, Resistor_SMD:R_0805_2012Metric_Pad1.15x1.40mm_HandSolder, symbol Device:R
- removed R13, R17: 27k, Resistor_SMD:R_0805_2012Metric_Pad1.15x1.40mm_HandSolder, symbol Device:R
- removed R14: 100k, Resistor_SMD:R_0805_2012Metric_Pad1.15x1.40mm_HandSolder, symbol Device:R
- removed R15, R16, R35, R42: 22k, Resistor_SMD:R_0805_2012Metric_Pad1.15x1.40mm_HandSolder, symbol Device:R
- removed R18, R19, R23, R24, R38: 10K, Resistor_SMD:R_0805_2012Metric_Pad1.15x1.40mm_HandSolder, symbol Device:R
- removed R2: 560, Resistor_SMD:R_0805_2012Metric_Pad1.15x1.40mm_HandSolder, symbol Device:R
- removed R21, R60: 1.8k, Resistor_SMD:R_0805_2012Metric_Pad1.15x1.40mm_HandSolder, symbol Device:R
- removed R25, R26, R27, R28: 3.9k, Resistor_SMD:R_0805_2012Metric_Pad1.15x1.40mm_HandSolder, symbol Device:R
- removed R29, R59: 1k, Resistor_SMD:R_0805_2012Metric_Pad1.15x1.40mm_HandSolder, symbol Device:R
- removed R30, R33, R34: 100, Resistor_SMD:R_1206_3216Metric_Pad1.42x1.75mm_HandSolder, symbol Device:R
- removed R36: 12k, Resistor_SMD:R_0805_2012Metric_Pad1.15x1.40mm_HandSolder, symbol Device:R
- removed R37, R40, R41, R62, R63: 2.2K, Resistor_SMD:R_0805_2012Metric_Pad1.15x1.40mm_HandSolder, symbol Device:R
- removed R4: 2.7K, Resistor_SMD:R_0805_2012Metric_Pad1.15x1.40mm_HandSolder, symbol Device:R
- removed R43: 4.7k, Resistor_SMD:R_0805_2012Metric_Pad1.15x1.40mm_HandSolder, symbol Device:R
- removed R44, R45: 220, Resistor_SMD:R_1206_3216Metric_Pad1.42x1.75mm_HandSolder, symbol Device:R
- removed R46, R47, R50, R51: 5.6K, Resistor_SMD:R_0805_2012Metric_Pad1.15x1.40mm_HandSolder, symbol Device:R
- removed R49: 10 1W, Resistor_THT:R_Axial_DIN0411_L9.9mm_D3.6mm_P12.70mm_Horizontal, symbol Device:R
- removed R53, R55, R57: 6.8k, Resistor_SMD:R_0805_2012Metric_Pad1.15x1.40mm_HandSolder, symbol Device:R
- removed R54, R7: 1.8K, Resistor_SMD:R_0805_2012Metric_Pad1.15x1.40mm_HandSolder, symbol Device:R
- removed R56, R58: 6.8K, Resistor_SMD:R_0805_2012Metric_Pad1.15x1.40mm_HandSolder, symbol Device:R
- removed R61, R65: 82k, Resistor_SMD:R_0805_2012Metric_Pad1.15x1.40mm_HandSolder, symbol Device:R
- removed RV1: 10K linear (gain), Connector_PinHeader_2.54mm:PinHeader_2x03_P2.54mm_Vertical, symbol Device:R_POT_Dual
- removed RV2: 1K log (headphone vol), Connector_PinHeader_2.54mm:PinHeader_2x03_P2.54mm_Vertical, symbol Device:R_POT_Dual
- removed RV3: 10k (SEND_LEVEL), Connector_PinHeader_2.54mm:PinHeader_1x03_P2.54mm_Vertical, symbol Device:R_POT
- removed RV4: 10k linear (FREQUENCY), Project-152-Bass-Guitar-Amp.pretty:RM-065-TRIMPOT, symbol Device:R_POT
- removed RV5: 10k linear (BALANCE), Project-152-Bass-Guitar-Amp.pretty:RM-065-TRIMPOT, symbol Device:R_POT
- removed SW1: SW_DPST, Connector_PinHeader_2.54mm:PinHeader_2x02_P2.54mm_Vertical, symbol Switch:SW_DPST
- removed SW2: SW_SPDT, Connector_PinHeader_2.54mm:PinHeader_1x03_P2.54mm_Vertical, symbol Switch:SW_SPDT
- removed SW3: GND LIFT, Connector_PinHeader_2.54mm:PinHeader_1x02_P2.54mm_Vertical, symbol Switch:SW_SPST
- removed SW4: SW_SPST, Connector_PinHeader_2.54mm:PinHeader_1x02_P2.54mm_Vertical, symbol Switch:SW_SPST
- removed SW5: SW_HPFQ, Connector_PinHeader_2.54mm:PinHeader_2x02_P2.54mm_Vertical, symbol Switch:SW_DPST
- removed U1: OPA2134, Package_DIP:DIP-8_W7.62mm_Socket, symbol Amplifier_Operational:TL072
- removed U2, U3, U4, U6, U7, U8, U9: NE5532, Package_DIP:DIP-8_W7.62mm_Socket, symbol Amplifier_Operational:NE5532
- removed U5: TL072, Package_DIP:DIP-8_W7.62mm_Socket, symbol Amplifier_Operational:TL072
Other:
- note removed: "(EQ board is separate)"
- note removed: "Crossover"
- note removed: "DI out"
- note removed: "EFX"
- note removed: "Frequency Switch (27hz or 37hz)"
- note removed: "GAIN SW"
- note removed: "Gain Sw"
- note removed: "Headphone Amplifier"
- note removed: "Hi-pass filter Bypass\n"
- note removed: "High-pass filter to remove subsonic frequencies"
- note removed: "Initial Gain Stage"
- note removed: "Input from MP3 player, etc."
- note removed: "Output to headphones"
- note removed: "Overload indicator"
- note removed: "Power"
- note removed: "Ring"
- note removed: "Tip"
- note removed: "Tip Switch"
- note removed: "To 1/4" jack"
- note removed: "To Eq"
- note removed: "To the Power Amp"
- note removed: "Tuner Out"

Commit message: Did some layout
Parts:
- added C1, C2: 1uF, Capacitor_THT:C_Rect_L7.2mm_W7.2mm_P5.00mm_FKS2_FKP2_MKS2_MKP2, symbol Device:C
- added C10, C11, C17: 100uF 50V, Capacitor_THT:CP_Radial_D8.0mm_P3.50mm, symbol Device:CP
- added C12, C13, C15, C16, C18, C19, C20, C21, C22, C23, C24, C25, C26, C27, C28, C30, C31, C33, C36, C37: 0.1uF, Capacitor_SMD:C_0805_2012Metric_Pad1.15x1.40mm_HandSolder, symbol Device:C
- added C14: 100uF 50V, Capacitor_THT:CP_Radial_D8.0mm_P2.50mm, symbol Device:CP
- added C29: 0.1uF (AUDIO), Capacitor_THT:C_Rect_L7.2mm_W2.5mm_P5.00mm_FKS2_FKP2_MKS2_MKP2, symbol Device:C
- added C3, C6, C7, C9: 120n, Capacitor_THT:C_Rect_L7.2mm_W3.5mm_P5.00mm_FKS2_FKP2_MKS2_MKP2, symbol Device:C
- added C32, C34, C35: 15nF, Capacitor_THT:C_Rect_L7.2mm_W2.5mm_P5.00mm_FKS2_FKP2_MKS2_MKP2, symbol Device:C
- added C4: 47uF 63V, Capacitor_THT:CP_Radial_D8.0mm_P5.00mm, symbol Device:CP
- added C41, C42, C43, C44: 100uF 63V, Capacitor_THT:CP_Radial_D8.0mm_P3.50mm, symbol Device:CP
- added C5: 10uF 50V, Capacitor_THT:CP_Radial_D6.3mm_P2.50mm, symbol Device:CP
- added D10, D11, D2, D3, D4, D5, D6, D7: 1N4148, Diode_THT:D_DO-35_SOD27_P7.62mm_Horizontal, symbol Diode:1N4148
- added D12: OVERLOAD, LED_THT:LED_D3.0mm, symbol Device:LED
- added D13: POWER, LED_THT:LED_D3.0mm, symbol Device:LED
- added D14, D15, D16, D17: 10V, Diode_THT:D_DO-41_SOD81_P7.62mm_Horizontal, symbol Device:D_Zener
- added J1, J4, J5: Conn_01x03_Male, Connector_PinHeader_2.54mm:PinHeader_1x03_P2.54mm_Vertical, symbol Connector:Conn_01x03_Male
- added J12: XLR3, Connector_PinHeader_2.54mm:PinHeader_1x03_P2.54mm_Vertical, symbol Connector:XLR3
- added J14: Conn_01x03, Connector_PinHeader_2.54mm:PinHeader_1x03_P2.54mm_Vertical, symbol Connector_Generic:Conn_01x03
- added J15, J16, J17: Conn_01x02, Connector_PinHeader_2.54mm:PinHeader_1x02_P2.54mm_Vertical, symbol Connector_Generic:Conn_01x02
- added J2, J3, J6: Conn_01x02_Male, Connector_PinHeader_2.54mm:PinHeader_1x02_P2.54mm_Vertical, symbol Connector:Conn_01x02_Male
- added J7: Conn_01x03, TerminalBlock_Phoenix:TerminalBlock_Phoenix_MKDS-1,5-3_1x03_P5.00mm_Horizontal, symbol Connector_Generic:Conn_01x03
- added J8: Conn_01x05_Female, Connector_PinHeader_2.54mm:PinHeader_1x05_P2.54mm_Vertical, symbol Connector:Conn_01x05_Female
- added Q1, Q3: 2N3904, Package_TO_SOT_THT:TO-92_Inline, symbol Transistor_BJT:2N3904
- added Q2, Q4: 2N3906, Package_TO_SOT_THT:TO-92_Inline, symbol Transistor_BJT:2N3906
- added Q5: BC549, Package_TO_SOT_THT:TO-92_Inline, symbol Transistor_BJT:BC549
- added R1, R39: 1M, Resistor_SMD:R_0805_2012Metric_Pad1.15x1.40mm_HandSolder, symbol Device:R
- added R10, R11, R20, R22, R3, R31, R32, R48, R5, R52, R6, R8, R9: 10k, Resistor_SMD:R_0805_2012Metric_Pad1.15x1.40mm_HandSolder, symbol Device:R
- added R12, R64: 33k, Resistor_SMD:R_0805_2012Metric_Pad1.15x1.40mm_HandSolder, symbol Device:R
- added R13, R17: 27k, Resistor_SMD:R_0805_2012Metric_Pad1.15x1.40mm_HandSolder, symbol Device:R
- added R14: 100k, Resistor_SMD:R_0805_2012Metric_Pad1.15x1.40mm_HandSolder, symbol Device:R
- added R15, R16, R35, R42: 22k, Resistor_SMD:R_0805_2012Metric_Pad1.15x1.40mm_HandSolder, symbol Device:R
- added R18, R19, R23, R24, R38: 10K, Resistor_SMD:R_0805_2012Metric_Pad1.15x1.40mm_HandSolder, symbol Device:R
- added R2: 560, Resistor_SMD:R_0805_2012Metric_Pad1.15x1.40mm_HandSolder, symbol Device:R
- added R21, R60: 1.8k, Resistor_SMD:R_0805_2012Metric_Pad1.15x1.40mm_HandSolder, symbol Device:R
- added R25, R26, R27, R28: 3.9k, Resistor_SMD:R_0805_2012Metric_Pad1.15x1.40mm_HandSolder, symbol Device:R
- added R29, R59: 1k, Resistor_SMD:R_0805_2012Metric_Pad1.15x1.40mm_HandSolder, symbol Device:R
- added R30, R33, R34: 100, Resistor_SMD:R_1206_3216Metric_Pad1.42x1.75mm_HandSolder, symbol Device:R
- added R36: 12k, Resistor_SMD:R_0805_2012Metric_Pad1.15x1.40mm_HandSolder, symbol Device:R
- added R37, R40, R41, R62, R63: 2.2K, Resistor_SMD:R_0805_2012Metric_Pad1.15x1.40mm_HandSolder, symbol Device:R
- added R4: 2.7K, Resistor_SMD:R_0805_2012Metric_Pad1.15x1.40mm_HandSolder, symbol Device:R
- added R43: 4.7k, Resistor_SMD:R_0805_2012Metric_Pad1.15x1.40mm_HandSolder, symbol Device:R
- added R44, R45: 220, Resistor_SMD:R_1206_3216Metric_Pad1.42x1.75mm_HandSolder, symbol Device:R
- added R46, R47, R50, R51: 5.6K, Resistor_SMD:R_0805_2012Metric_Pad1.15x1.40mm_HandSolder, symbol Device:R
- added R49: 10 1W, Resistor_THT:R_Axial_DIN0411_L9.9mm_D3.6mm_P12.70mm_Horizontal, symbol Device:R
- added R53, R55, R57: 6.8k, Resistor_SMD:R_0805_2012Metric_Pad1.15x1.40mm_HandSolder, symbol Device:R
- added R54, R7: 1.8K, Resistor_SMD:R_0805_2012Metric_Pad1.15x1.40mm_HandSolder, symbol Device:R
- added R56, R58: 6.8K, Resistor_SMD:R_0805_2012Metric_Pad1.15x1.40mm_HandSolder, symbol Device:R
- added R61, R65: 82k, Resistor_SMD:R_0805_2012Metric_Pad1.15x1.40mm_HandSolder, symbol Device:R
- added RV1: 10K linear (gain), Connector_PinHeader_2.54mm:PinHeader_2x03_P2.54mm_Vertical, symbol Device:R_POT_Dual
- added RV2: 1K log (headphone vol), Connector_PinHeader_2.54mm:PinHeader_2x03_P2.54mm_Vertical, symbol Device:R_POT_Dual
- added RV3: 10k (SEND_LEVEL), Connector_PinHeader_2.54mm:PinHeader_1x03_P2.54mm_Vertical, symbol Device:R_POT
- added RV4: 10k linear (FREQUENCY), Connector_PinHeader_2.54mm:PinHeader_1x03_P2.54mm_Vertical, symbol Device:R_POT
- added RV5: 10k linear (BALANCE), Connector_PinHeader_2.54mm:PinHeader_1x03_P2.54mm_Vertical, symbol Device:R_POT
- added SW1: SW_DPST, Connector_PinHeader_2.54mm:PinHeader_2x02_P2.54mm_Vertical, symbol Switch:SW_DPST
- added SW2: SW_SPDT, Connector_PinHeader_2.54mm:PinHeader_1x03_P2.54mm_Vertical, symbol Switch:SW_SPDT
- added SW3: GND LIFT, Connector_PinHeader_2.54mm:PinHeader_1x02_P2.54mm_Vertical, symbol Switch:SW_SPST
- added SW4: SW_SPST, Connector_PinHeader_2.54mm:PinHeader_1x02_P2.54mm_Vertical, symbol Switch:SW_SPST
- added SW5: SW_HPFQ, Connector_PinHeader_2.54mm:PinHeader_2x02_P2.54mm_Vertical, symbol Switch:SW_DPST
- added U1: OPA2134, Package_DIP:DIP-8_W7.62mm_Socket, symbol Amplifier_Operational:TL072
- added U2, U3, U4, U6, U7, U8, U9: NE5532, Package_DIP:DIP-8_W7.62mm_Socket, symbol Amplifier_Operational:NE5532
- added U5: TL072, Package_DIP:DIP-8_W7.62mm_Socket, symbol Amplifier_Operational:TL072
Connections:
- new net: R4.1, R6.1, R7.1, U1.2 (-)
- new net: C4.1, R7.2
- new net: C4.2, R14.1, SW4.1 (A)
- new net: C5.2, D2.2 (A), RV1.1
- new net: R20.1, RV1.2, U1.5 (+)
- new net: C5.1, R6.2, U1.1
- new net: R2.1, U1.3 (+)
- new net: R21.1, R22.2, U1.6 (-)
- new net: C10.1, R22.1, U1.7
- new net: J2.2 (Pin_2), R1.2, R2.2
- new net: C17.2, R31.1, R33.2
- new net: R18.2, R23.1, U3.6 (-)
- new net: D3.1 (K), D4.2 (A), R23.2, U3.7
- new net: R15.2, R18.1, U3.1
- new net: R15.1, R8.2, R9.2, U3.2 (-)
- new net: C7.2, R13.1, SW1.2, SW5.3, U2.1, U2.2 (-)
- new net: C6.1, R61.1, SW1.4, U2.3 (+)
- new net: C9.1, R65.1, SW1.1, U2.5 (+)
- new net: C11.1, R17.1, R64.1, U2.6 (-), U2.7
- new net: C3.1, C6.2, R12.2, R13.2
- new net: C2.1, R10.1
- new net: R10.2, R11.2, R16.1, U4.2 (-)
- new net: C1.1, R9.1
- new net: D13.2 (A), R48.2
- new net: D12.2 (A), R43.2
- new net: C7.1, C9.2, R17.2, SW5.1
- new net: D10.2 (A), U5.1
- new net: R35.2, R36.1, U5.2 (-)
- new net: U5.6 (-), U5.7
- new net: C11.2, R30.2
- new net: C22.2, D10.1 (K), Q5.2 (B)
- new net: C14.1, Q3.1 (E), Q4.3 (C)
- new net: D5.2 (A), Q3.2 (B), R27.2
- new net: D6.1 (K), Q4.2 (B), R28.1
- new net: D5.1 (K), D6.2 (A), R24.2, U4.7
- new net: R19.2, R24.1, U4.6 (-)
- new net: R16.2, R19.1, U4.1
- new net: C17.1, Q1.1 (E), Q2.3 (C)
- new net: D3.2 (A), Q1.2 (B), R25.2
- new net: D4.1 (K), Q2.2 (B), R26.1
- new net: R33.1, RV2.1
- new net: R34.1, RV2.4
- new net: C14.2, R32.1, R34.2
- new net: Q5.3 (E), R43.1
- new net: C2.2, J1.3 (Pin_3), R3.1
- new net: C1.2, J1.2 (Pin_2), R5.1
- new net: D11.2 (A), D14.2 (A), R41.1, R45.2, R62.2, U6.1
- new net: R40.2, R41.2, U6.2 (-)
- new net: R38.2, RV3.2, U6.3 (+)
- new net: R62.1, R63.2, U6.6 (-)
- new net: D16.2 (A), R44.2, R63.1, U6.7
- new net: C33.2, J12.1, R49.1
- new net: C44.1, J12.2
- new net: C43.1, J12.3
- new net: R49.2, SW3.2 (B)
- new net: RV3.1, SW2.2 (B)
- new net: R37.2, RV3.3
- new net: C41.1, R44.1
- new net: C42.1, R45.1
- new net: J5.3 (Pin_3), RV2.2
- new net: J5.2 (Pin_2), RV2.5
- new net: R64.2, SW5.2
- new net: R12.1, SW5.4
- new net: D16.1 (K), D17.1 (K)
- new net: R46.2, R47.1, U8.3 (+)
- new net: C29.1, R47.2, R58.2, U8.7
- new net: R50.1, R54.1, R56.2, U8.1
- new net: R50.2, R51.1, U8.2 (-)
- new net: D14.1 (K), D15.1 (K)
- new net: R54.2, RV4.3
- new net: C29.2, RV4.1, RV4.2, U8.6 (-)
- new net: C41.2, C43.2
- new net: C42.2, C44.2
- new net: C35.2, R57.1, U9.5 (+)
- new net: R52.1, R55.1, R59.1, U9.7
- new net: C23.1, C24.2
- new net: C32.2, C34.1, R52.2, R53.1
- new net: C34.2, C35.1, R55.2
- new net +12V: C12.2, C15.2, C18.2, C20.2, C23.2, C25.2, C27.2, C30.2, C36.2, J7.1 (Pin_1), J8.2 (Pin_2), Q1.3 (C), Q3.3 (C), Q5.1 (C), R25.1, R27.1, R35.1, R48.1, U1.8 (V+), U2.8 (V+), U3.8 (V+), U4.8 (V+), U5.8 (V+), U6.8 (V+), U7.8 (V+), U8.8 (V+), U9.8 (V+)
- new net -12V: C13.1, C16.1, C19.1, C21.1, C24.1, C26.1, C28.1, C31.1, C37.1, D13.1 (K), J7.3 (Pin_3), J8.3 (Pin_3), Q2.1 (E), Q4.1 (E), R26.2, R28.2, U1.4 (V-), U2.4 (V-), U3.4 (V-), U4.4 (V-), U6.4 (V-), U7.4 (V-), U8.4 (V-), U9.4 (V-)
- new net EFXreturn: J4.3 (Pin_3), R11.1, R8.1, SW2.1 (A)
- new net EFXsend: J3.2 (Pin_2), J4.2 (Pin_2), R30.1
- new net FromEQ: C3.2, J8.5 (Pin_5), R42.2, SW1.3, U7.3 (+)
- new net GND: C12.1, C13.2, C15.1, C16.2, C18.1, C19.2, C20.1, C21.2, C25.1, C26.2, C27.1, C28.2, C33.1, C36.1, C37.2, D15.2 (A), D17.2 (A), J1.1 (Pin_1), J14.1 (Pin_1), J15.1 (Pin_1), J16.1 (Pin_1), J17.1 (Pin_1), J2.1 (Pin_1), J3.1 (Pin_1), J4.1 (Pin_1), J5.1 (Pin_1), J6.1 (Pin_1), J7.2 (Pin_2), J8.1 (Pin_1), R1.1, R14.2, R20.2, R21.2, R3.2, R31.2, R32.2, R37.1, R38.1, R4.2, R40.1, R42.1, R5.2, R51.2, R53.2, R57.2, R60.2, R61.2, R65.2, RV1.3, RV1.6, RV2.3, RV2.6, RV5.2, SW3.1 (A), SW4.2 (B), U3.3 (+), U3.5 (+), U4.3 (+), U4.5 (+), U6.5 (+), U8.5 (+)
- new net GNDD: C22.1, C30.1, C31.2, D12.1 (K), R36.2, R39.2, U5.4 (V-), U5.5 (+)
- new net HF: J14.2 (Pin_2), J15.2 (Pin_2), U9.1, U9.2 (-)
- new net HF*: R56.1, RV5.3, U9.3 (+)
- new net LF: J14.3 (Pin_3), U7.6 (-), U7.7
- new net LF*: R58.1, RV5.1, U7.5 (+)
- new net Overload: D11.1 (K), D2.1 (K), D7.1 (K), R39.1, U5.3 (+)
- new net PreEQ: C10.2, D7.2 (A), R29.2, RV1.4, SW2.3 (C)
- new net ToEQ: J8.4 (Pin_4), RV1.5
- new net Tuner: J6.2 (Pin_2), R29.1
- new net Tweeter: J17.2 (Pin_2), R59.2, R60.1, U9.6 (-)
- new net TweeterXOVR: C32.1, R46.1, U7.1, U7.2 (-)
Other:
- note added: "(EQ board is separate)"
- note added: "Crossover"
- note added: "DI out"
- note added: "EFX"
- note added: "Frequency Switch (27hz or 37hz)"
- note added: "GAIN SW"
- note added: "Gain Sw"
- note added: "Headphone Amplifier"
- note added: "Hi-pass filter Bypass\n"
- note added: "High-pass filter to remove subsonic frequencies"
- note added: "Initial Gain Stage"
- note added: "Input from MP3 player, etc."
- note added: "Output to headphones"
- note added: "Overload indicator"
- note added: "Power"
- note added: "Ring"
- note added: "Tip"
- note added: "Tip Switch"
- note added: "To 1/4" jack"
- note added: "To Eq"
- note added: "To the Power Amp"
- note added: "Tuner Out"

Commit message: More layout work
Also fixed some minor issues on the schematic
Connections:
- net EFXreturn: now also R42.2, U7.3 (+)
- net FromEQ: no longer R42.2, U7.3 (+)
- net GND: now also C23.1, C24.2
- net LF: now also J16.2 (Pin_2)
Changed lines of the file:
@@
 Wire Wire Line
 	12650 7850 12900 7850
-Text GLabel 12650 7850 0    50   Input ~ 0
-FromEQ
 $Comp
 L Device:R R42
@@
 Wire Wire Line
 	4150 1050 4150 1200
+Text GLabel 12650 7850 0    50   Input ~ 0
+EFXreturn
+Wire Wire Line
+	18800 14200 18850 14200
+$Comp
+L power:GND #PWR?
+U 1 1 5E7B6FD0
+P 12500 9700
+F 0 "#PWR?" H 12500 9450 50  0001 C CNN
+F 1 "GND" H 12505 9527 50  0000 C CNN
+F 2 "" H 12500 9700 50  0001 C CNN
+F 3 "" H 12500 9700 50  0001 C CNN
+	1    12500 9700
+	1    0    0    -1
+$EndComp
 $EndSCHEMATC

Commit message: More layout progress
Parts:
- RV5: footprint Connector_PinHeader_2.54mm:PinHeader_1x03_P2.54mm_Vertical -> Project-152-Bass-Guitar-Amp.pretty:RM-065-TRIMPOT
Changed lines of the file:
@@
 F 0 "RV5" H 17830 8546 50  0000 R CNN
 F 1 "10k linear (BALANCE)" H 17830 8455 50  0000 R CNN
-F 2 "Connector_PinHeader_2.54mm:PinHeader_1x03_P2.54mm_Vertical" H 17900 8500 50  0001 C CNN
+F 2 "Project-152-Bass-Guitar-Amp.pretty:RM-065-TRIMPOT" H 17900 8500 50  0001 C CNN
 F 3 "~" H 17900 8500 50  0001 C CNN
 	1    17900 8500
@@
 	18800 14200 18850 14200
 $Comp
-L power:GND #PWR?
+L power:GND #PWR0103
 U 1 1 5E7B6FD0
 P 12500 9700
-F 0 "#PWR?" H 12500 9450 50  0001 C CNN
+F 0 "#PWR0103" H 12500 9450 50  0001 C CNN
 F 1 "GND" H 12505 9527 50  0000 C CNN
 F 2 "" H 12500 9700 50  0001 C CNN

Commit message: Did more layout work
Parts:
- RV4: footprint Connector_PinHeader_2.54mm:PinHeader_1x03_P2.54mm_Vertical -> Project-152-Bass-Guitar-Amp.pretty:RM-065-TRIMPOT
Changed lines of the file:
@@
 F 0 "RV4" H 15980 10046 50  0000 R CNN
 F 1 "10k linear (FREQUENCY)" H 15980 9955 50  0000 R CNN
-F 2 "Connector_PinHeader_2.54mm:PinHeader_1x03_P2.54mm_Vertical" H 16050 10000 50  0001 C CNN
+F 2 "Project-152-Bass-Guitar-Amp.pretty:RM-065-TRIMPOT" H 16050 10000 50  0001 C CNN
 F 3 "~" H 16050 10000 50  0001 C CNN
 	1    16050 10000
