File: Preamp/Preamplifier.kicad_pcb (KiCad board)
At the start: 2 copper layers, 200 x 95 mm, 165 parts, among them J1 Conn_01x02_Female, J10 AudioJack2, J11 Conn_01x05_Female, J12 XLR3, J13 Conn_01x03, J14 Conn_01x03, J15 Conn_01x02, J16 Conn_01x02, J17 Conn_01x02, J2 AudioJack2, J3 AudioJack3_SwitchTR, J4 AudioJack2_SwitchT, J5 AudioJack2_SwitchT, J6 Conn_01x02_Male, J7 Conn_01x02_Male, J8 Conn_01x05_Female, J9 AudioJack3_SwitchTR, Q1 2N3904, Q2 2N3906, Q3 2N3904, Q4 2N3906, Q5 BC549, SW1 SW_DPST, SW2 SW_SPDT, SW3 GND LIFT, SW4 SW_SPST, T1 Transformer_1P_2S, U1 OPA2134, U2 NE5532, U3 NE5532, U4 NE5532, U5 TL072, U6 NE5532, U7 NE5532, U8 NE5532, U9 NE5532

Commit message: Did some layout
Parts:
- removed C38, C39, C40, C8: 1000uF 50V, Capacitor_THT:CP_Radial_D17.0mm_P7.50mm
- removed D8, D9: 1N5819, Diode_THT:D_DO-41_SOD81_P10.16mm_Horizontal
- removed F1: Fuse, Fuse:Fuseholder_Cylinder-5x20mm_Schurter_0031-8002_Horizontal_Open
- removed J10: AudioJack2, TerminalBlock_Phoenix:TerminalBlock_Phoenix_PT-1,5-2-3.5-H_1x02_P3.50mm_Horizontal
- removed J11: Conn_01x05_Female, TerminalBlock_Phoenix:TerminalBlock_Phoenix_PT-1,5-5-3.5-H_1x05_P3.50mm_Horizontal
- removed J13: Conn_01x03, TerminalBlock_Phoenix:TerminalBlock_Phoenix_PT-1,5-3-3.5-H_1x03_P3.50mm_Horizontal
- removed J9: AudioJack3_SwitchTR, TerminalBlock_Phoenix:TerminalBlock_Phoenix_PT-1,5-5-3.5-H_1x05_P3.50mm_Horizontal
- removed T1: Transformer_1P_2S, Project-152-Bass-Guitar-Amp:TE 49008024RC62
- added R64: 33k, Resistor_SMD:R_0805_2012Metric_Pad1.15x1.40mm_HandSolder, F.Cu at (403.3, 143.7)
- added R65: 82k, Resistor_SMD:R_0805_2012Metric_Pad1.15x1.40mm_HandSolder, F.Cu at (417.4, 136.7)
- added SW5: SW_HPFQ, Connector_PinHeader_2.54mm:PinHeader_2x02_P2.54mm_Vertical, F.Cu at (380.5, 140.1)
- D12: footprint Connector_Phoenix_MSTB:PhoenixContact_MSTBA_2,5_2-G_1x02_P5.00mm_Horizontal -> LED_THT:LED_D3.0mm
- D13: footprint Connector_Phoenix_MSTB:PhoenixContact_MSTBA_2,5_2-G-5,08_1x02_P5.08mm_Horizontal -> LED_THT:LED_D3.0mm
- J1: value Conn_01x02_Female -> Conn_01x03_Male; footprint TerminalBlock_Dinkle:TerminalBlock_Dinkle_DT-55-B01X-02_P10.00mm -> Connector_PinHeader_2.54mm:PinHeader_1x03_P2.54mm_Vertical
- J12, J14, RV3, RV4, RV5, SW2: footprint TerminalBlock_Phoenix:TerminalBlock_Phoenix_PT-1,5-3-3.5-H_1x03_P3.50mm_Horizontal -> Connector_PinHeader_2.54mm:PinHeader_1x03_P2.54mm_Vertical
- J15, J16, J17, SW4: footprint TerminalBlock_Phoenix:TerminalBlock_Phoenix_PT-1,5-2-3.5-H_1x02_P3.50mm_Horizontal -> Connector_PinHeader_2.54mm:PinHeader_1x02_P2.54mm_Vertical
- J2: value AudioJack2 -> Conn_01x02_Male; footprint TerminalBlock_Phoenix:TerminalBlock_Phoenix_PT-1,5-2-3.5-H_1x02_P3.50mm_Horizontal -> Connector_PinHeader_2.54mm:PinHeader_1x02_P2.54mm_Vertical
- J3: value AudioJack3_SwitchTR -> Conn_01x02_Male; footprint TerminalBlock_Phoenix:TerminalBlock_Phoenix_PT-1,5-5-3.5-H_1x05_P3.50mm_Horizontal -> Connector_PinHeader_2.54mm:PinHeader_1x02_P2.54mm_Vertical
- J4, J5: value AudioJack2_SwitchT -> Conn_01x03_Male; footprint TerminalBlock_Phoenix:TerminalBlock_Phoenix_PT-1,5-3-3.5-H_1x03_P3.50mm_Horizontal -> Connector_PinHeader_2.54mm:PinHeader_1x03_P2.54mm_Vertical
- J6: footprint TerminalBlock_Phoenix:TerminalBlock_Phoenix_PT-1,5-2-5.0-H_1x02_P5.00mm_Horizontal -> Connector_PinHeader_2.54mm:PinHeader_1x02_P2.54mm_Vertical
- J7: value Conn_01x02_Male -> Conn_01x03; footprint TerminalBlock_Phoenix:TerminalBlock_Phoenix_PT-1,5-2-5.0-H_1x02_P5.00mm_Horizontal -> TerminalBlock_Phoenix:TerminalBlock_Phoenix_MKDS-1,5-3_1x03_P5.00mm_Horizontal
- J8: footprint TerminalBlock_Phoenix:TerminalBlock_Phoenix_PT-1,5-5-3.5-H_1x05_P3.50mm_Horizontal -> Connector_PinHeader_2.54mm:PinHeader_1x05_P2.54mm_Vertical
- R1, R14, R62: moved to B.Cu
- R12: value 0 -> 33k; footprint Resistor_THT:R_Axial_DIN0207_L6.3mm_D2.5mm_P10.16mm_Horizontal -> Resistor_SMD:R_0805_2012Metric_Pad1.15x1.40mm_HandSolder
- R49: footprint Resistor_THT:R_Axial_DIN0411_L9.9mm_D3.6mm_P25.40mm_Horizontal -> Resistor_THT:R_Axial_DIN0411_L9.9mm_D3.6mm_P12.70mm_Horizontal
- R60: value 1k -> 1.8k
- RV1, RV2: footprint TerminalBlock_Phoenix:TerminalBlock_Phoenix_PT-1,5-6-3.5-H_1x06_P3.50mm_Horizontal -> Connector_PinHeader_2.54mm:PinHeader_2x03_P2.54mm_Vertical
- SW1: footprint TerminalBlock_Phoenix:TerminalBlock_Phoenix_PT-1,5-4-3.5-H_1x04_P3.50mm_Horizontal -> Connector_PinHeader_2.54mm:PinHeader_2x02_P2.54mm_Vertical
- SW3: footprint TerminalBlock_Phoenix:TerminalBlock_Phoenix_MKDS-3-2-5.08_1x02_P5.08mm_Horizontal -> Connector_PinHeader_2.54mm:PinHeader_1x02_P2.54mm_Vertical
- moved J7 504.1 mm to (3.50, 6.00)
- moved J6 473.4 mm to (18.8, 2.25), turned to 90 degrees
- moved J16 464.5 mm to (47.7, -15.1), turned to 90 degrees
- moved J17 462.1 mm to (37.3, -24.2)
- moved J15 457.2 mm to (56.9, -14.7), turned to 90 degrees
- moved C43 454.6 mm to (43.6, 8.80), turned to 270 degrees
- moved J12 450.3 mm to (35.6, 2.30), turned to 90 degrees
- moved C44 447.6 mm to (34.6, 8.80), turned to 270 degrees
- moved C41 442.3 mm to (43.6, 21.8), turned to 90 degrees
- moved C42 436.3 mm to (34.6, 21.8), turned to 90 degrees
- moved R6 404.6 mm to (4.50, 76.5), turned to 90 degrees
- moved R2 401.7 mm to (5.40, 95.6), turned to 270 degrees
- moved R49 400.0 mm to (26.9, 2.30), turned to 270 degrees
- moved J14 396.6 mm to (67.5, -11.7), turned to 90 degrees
- moved RV2 393.3 mm to (37.5, 97.0), turned to 90 degrees
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Connections:
- J1 pad 1: Net-(J1-Pad1) -> GND
- J1 pad 2: Net-(F1-Pad2) -> Net-(C1-Pad2)
- J14 pad 1: HF -> GND
- J14 pad 2: LF -> HF
- J14 pad 3: GND -> LF
- J15 pad 1: HF -> GND
- J15 pad 2: GND -> HF
- J16 pad 1: LF -> GND
- J16 pad 2: GND -> (no net)
- J17 pad 1: Tweeter -> GND
- J17 pad 2: GND -> Tweeter
- J2 pad 1: (no net) -> GND
- J2 pad 2: (no net) -> Net-(J2-Pad2)
- J3 pad 1: (no net) -> GND
- J3 pad 2: (no net) -> EFXsend
- J4 pad 1: (no net) -> GND
- J4 pad 2: (no net) -> EFXsend
- J4 pad 3: (no net) -> EFXreturn
- J5 pad 1: (no net) -> GND
- J5 pad 2: (no net) -> Net-(J5-Pad2)
- J5 pad 3: (no net) -> Net-(J5-Pad3)
- J6 pad 1: (no net) -> GND
- J6 pad 2: (no net) -> Tuner
- J7 pad 1: (no net) -> +12V
- J7 pad 2: Net-(D9-Pad1) -> GND
- J8 pad 1: ToEQ -> GND
- J8 pad 2: FromEQ -> +12V
- J8 pad 3: +12V -> -12V
- J8 pad 4: GND -> ToEQ
- J8 pad 5: -12V -> FromEQ
- R1 pad 2: Net-(J2-PadT) -> Net-(J2-Pad2)
- R12 pad 1: GNDD -> Net-(R12-Pad1)
- R12 pad 2: GND -> Net-(C3-Pad1)
- R2 pad 2: Net-(J2-PadT) -> Net-(J2-Pad2)
- R29 pad 1: (no net) -> Tuner
- R30 pad 1: (no net) -> EFXsend
- R61 pad 1: FromEQ -> Net-(C6-Pad1)
- RV2 pad 2: (no net) -> Net-(J5-Pad3)
- RV2 pad 5: (no net) -> Net-(J5-Pad2)
Routing:
- net -12V: track 0.00 -> 106.9 mm, vias 0 -> 4
- net +12V: track 0.00 -> 89.5 mm
- net PreEQ: track 0.00 -> 27.2 mm
- net Net-(C5-Pad1): track 0.00 -> 24.2 mm, vias 0 -> 1
- net Net-(R2-Pad1): track 0.00 -> 20.0 mm, vias 0 -> 1
- net ToEQ: track 0.00 -> 17.3 mm
- net Net-(R20-Pad1): track 0.00 -> 14.8 mm
- net Net-(C5-Pad2): track 0.00 -> 13.3 mm, vias 0 -> 1
- net Net-(C10-Pad1): track 0.00 -> 10.5 mm
- net Net-(R4-Pad1): track 0.00 -> 10.2 mm
- net Net-(D11-Pad2): track 0.00 -> 8.04 mm
- net Net-(C44-Pad1): track 0.00 -> 7.97 mm
- net Net-(C43-Pad1): track 0.00 -> 7.71 mm
- net Net-(C4-Pad1): track 0.00 -> 7.53 mm
- net Net-(R40-Pad2): track 0.00 -> 7.14 mm
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- added copper zone on B.Cu, net GND
Other:
- board size 200 x 95 mm -> 100 x 100 mm
- net class Default: clearance 0.2 -> 0.25
- rule trace_clearance: 0.2 -> 0.25
- rule trace_min: 0.2 -> 0.25
- board text removed: "+12V"
- board text removed: "-12V"
- board text removed: "AUX IN"
- board text removed: "EFFECTS RETURN"
- board text removed: "FrEq"
- board text removed: "GAIN"
- board text removed: "GAIN SW"
- board text removed: "GND"
- board text removed: "GUITAR IN"
- board text removed: "TO EFFECTS"
- board text removed: "TO EQ BOARD"
- board text removed: "ToEq"
- board text removed: "WIP"

Commit message: More layout work
Also fixed some minor issues on the schematic
Parts:
- C13, C33, R45, R47: moved to B.Cu
- moved R45 397.8 mm to (15.7, 26.1), turned to 270 degrees
- moved R44 394.1 mm to (22.7, 27.1), turned to 270 degrees
- moved C37 391.4 mm to (10.7, 38.6), turned to 180 degrees
- moved C13 380.4 mm to (10.0, 82.0), turned to 90 degrees
- moved R42 375.1 mm to (47.7, 25.0), turned to 90 degrees
- moved C24 372.6 mm to (51.5, 29.3)
- moved R50 369.1 mm to (63.5, 20.0), turned to 270 degrees
- moved R46 368.4 mm to (63.5, 25.0), turned to 90 degrees
- moved R51 363.5 mm to (61.4, 20.0), turned to 90 degrees
- moved C27 363.2 mm to (73.0, 16.1)
- moved C23 362.0 mm to (57.1, 16.2)
- moved C12 361.1 mm to (14.0, 72.5)
- moved R56 360.5 mm to (67.4, 16.0), turned to 180 degrees
- moved D15 355.4 mm to (15.1, 18.0), turned to 180 degrees
- moved SW2 355.0 mm to (47.1, 96.8), turned to 270 degrees
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Connections:
- C23 pad 1: Net-(C23-Pad1) -> GND
- C24 pad 2: Net-(C23-Pad1) -> GND
- J16 pad 2: (no net) -> LF
- R42 pad 2: FromEQ -> EFXreturn
- U7 pad 3: FromEQ -> EFXreturn
Routing:
- net +12V: track 89.5 -> 137.6 mm, vias 0 -> 1
- net Net-(C33-Pad2): track 0.00 -> 35.0 mm
- net TweeterXOVR: track 0.00 -> 25.1 mm
- net EFXreturn: track 0.00 -> 24.6 mm
- net -12V: track 106.9 -> 128.4 mm
- net HF*: track 0.00 -> 21.3 mm
- net LF: track 0.00 -> 13.6 mm
- net Net-(C41-Pad1): track 0.00 -> 11.6 mm
- net Net-(C29-Pad1): track 0.00 -> 11.0 mm
- net Net-(D11-Pad2): track 8.04 -> 18.4 mm
- net Net-(C42-Pad1): track 0.00 -> 8.85 mm
- net Net-(C29-Pad2): track 0.00 -> 8.06 mm
- net Net-(R49-Pad2): track 0.00 -> 6.96 mm
- net Net-(D16-Pad2): track 2.71 -> 9.51 mm
- net Net-(R50-Pad1): track 0.00 -> 6.09 mm
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
Commit message: More layout progress
Parts:
- R13, R17, R58, R65: moved to B.Cu
- RV5: footprint Connector_PinHeader_2.54mm:PinHeader_1x03_P2.54mm_Vertical -> Project-152-Bass-Guitar-Amp.pretty:RM-065-TRIMPOT
- moved R58 357.7 mm to (67.4, 23.7)
- moved RV5 357.0 mm to (62.1, 8.60)
- moved R65 309.3 mm to (135.8, 8.80), turned to 90 degrees
- moved R17 304.1 mm to (135.8, 12.0), turned to 180 degrees
- moved C16 284.9 mm to (148.2, 7.00), turned to 180 degrees
- moved R13 278.3 mm to (157.8, 11.0)
- moved C9 275.9 mm to (138.2, 9.80), turned to 180 degrees
- moved C7 275.0 mm to (133.2, 14.0)
- moved C15 272.7 mm to (142.6, 20.2), turned to 180 degrees
- moved R12 269.2 mm to (161.6, 5.60), turned to 270 degrees
- moved C3 264.9 mm to (163.0, 8.60), turned to 270 degrees
- moved C6 254.7 mm to (158.8, 13.6), turned to 90 degrees
- moved U2 212.4 mm to (149.2, 17.4), turned to 180 degrees
- moved J17 10.3 mm to (87.6, 3.80)
- moved J14 8.09 mm to (70.4, 3.70)
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Routing:
- net +12V: track 137.6 -> 173.0 mm, vias 1 -> 2
- net LF*: track 0.00 -> 35.3 mm, vias 0 -> 2
- net LF: track 13.6 -> 34.3 mm
- net -12V: track 128.4 -> 148.4 mm
- net Net-(C7-Pad2): track 0.00 -> 17.4 mm
- net HF: track 5.00 -> 18.1 mm, vias 0 -> 1
- net Net-(C11-Pad1): track 0.00 -> 7.43 mm
- net Net-(C9-Pad1): track 0.00 -> 5.80 mm
- net Net-(C7-Pad1): track 0.00 -> 5.78 mm
- net Net-(R50-Pad1): track 6.09 -> 10.6 mm
- net EFXreturn: track 24.6 -> 20.1 mm, vias 0 -> 2
- net TweeterXOVR: track 25.1 -> 20.8 mm
- net GND: track 5.42 -> 9.27 mm, vias 14 -> 17
- net Tweeter: track 0.00 -> 2.90 mm
- net Net-(R46-Pad2): track 5.75 -> 6.43 mm
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
Commit message: Did more layout work
Parts:
- moved C24 4.07 mm to (45.8, 25.1), turned to 270 degrees
Routing:
- net -12V: track 148.4 -> 161.6 mm
- net LF: track 34.3 -> 35.6 mm

Commit message: More layout work
Parts:
- C23, C25, C27, R54, R57, R59, R60: moved to B.Cu
- RV4: footprint Connector_PinHeader_2.54mm:PinHeader_1x03_P2.54mm_Vertical -> Project-152-Bass-Guitar-Amp.pretty:RM-065-TRIMPOT
- moved R57 360.2 mm to (79.1, 24.1), turned to 180 degrees
- moved R53 352.6 mm to (83.0, 27.8), turned to 90 degrees
- moved R52 347.1 mm to (80.9, 27.8), turned to 270 degrees
- moved RV4 343.6 mm to (69.5, 8.55)
- moved R60 340.4 mm to (77.8, 20.2), turned to 90 degrees
- moved R55 339.6 mm to (78.8, 27.8), turned to 270 degrees
- moved C32 337.5 mm to (56.0, 27.2), turned to 270 degrees
- moved C34 288.9 mm to (59.2, 31.5)
- moved C35 280.0 mm to (67.2, 31.5)
- moved R54 25.7 mm to (69.8, 9.60), turned to 90 degrees
- moved R59 5.21 mm to (80.0, 20.2)
- moved J14 5.00 mm to (75.4, 3.70)
- moved C25 4.26 mm to (78.6, 16.7)
- moved J15 3.90 mm to (79.3, 3.70)
- moved C23 3.42 mm to (53.3, 16.6)
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Routing:
- net Net-(C29-Pad2): track 7.47 -> 32.1 mm
- net LF: track 35.6 -> 11.4 mm
- net Net-(C32-Pad2): track 0.00 -> 23.7 mm
- net Net-(C34-Pad2): track 0.00 -> 18.2 mm
- net Net-(C35-Pad2): track 0.00 -> 15.7 mm
- net Net-(R52-Pad1): track 3.06 -> 14.2 mm
- net GND: track 9.22 -> 5.42 mm, vias 17 -> 14
- net HF*: track 21.0 -> 24.6 mm, vias 0 -> 1
- net +12V: track 173.5 -> 170.3 mm
- net Net-(R50-Pad1): track 10.6 -> 13.6 mm, vias 0 -> 1
- net Net-(R54-Pad2): track 0.00 -> 2.26 mm
- net Tweeter: track 2.90 -> 4.67 mm
- net TweeterXOVR: track 20.8 -> 21.4 mm
- net HF: track 18.1 -> 18.6 mm, vias 1 -> 0

Commit message: Moar layout
Parts:
- C18, C19, C20, C21, R15, R19, R23, R24: moved to B.Cu
- moved J5 299.9 mm to (97.5, 97.2), turned to 270 degrees
- moved R15 296.7 mm to (134.6, 58.8), turned to 90 degrees
- moved C18 293.5 mm to (137.6, 57.2), turned to 270 degrees
- moved R23 287.6 mm to (137.5, 61.0), turned to 90 degrees
- moved C21 280.0 mm to (150.2, 64.2), turned to 90 degrees
- moved R18 275.5 mm to (132.9, 54.5)
- moved R11 270.3 mm to (148.8, 49.9), turned to 90 degrees
- moved R19 268.6 mm to (150.2, 58.4), turned to 270 degrees
- moved C20 261.7 mm to (153.2, 57.1), turned to 270 degrees
- moved R24 258.1 mm to (153.2, 61.0), turned to 90 degrees
- moved C19 257.7 mm to (134.6, 63.6), turned to 90 degrees
- moved R16 255.6 mm to (145.2, 58.6), turned to 90 degrees
- moved R10 252.1 mm to (151.0, 49.9), turned to 90 degrees
- moved U3 228.9 mm to (132.2, 57.3)
- moved U4 199.6 mm to (147.9, 57.4)
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Routing:
- net LF: track 11.4 -> 45.1 mm, vias 0 -> 1
- net GNDD: track 0.00 -> 7.62 mm
- net Net-(C32-Pad2): track 23.7 -> 30.3 mm
- net Net-(R19-Pad2): track 0.00 -> 6.59 mm
- net +12V: track 170.3 -> 175.6 mm
- net Net-(R16-Pad2): track 0.00 -> 5.08 mm
- net Net-(R10-Pad2): track 0.00 -> 2.83 mm
- net Net-(R15-Pad2): track 0.00 -> 2.60 mm
- net Net-(U5-Pad6): track 0.00 -> 2.54 mm
- net -12V: track 161.4 -> 163.9 mm
- net GND: track 5.42 -> 7.90 mm, vias 14 -> 13
- net Net-(R18-Pad2): track 0.00 -> 2.47 mm
- net Net-(C34-Pad2): track 18.2 -> 15.7 mm, vias 0 -> 1
- net Net-(R15-Pad1): track 0.00 -> 2.41 mm
- net Net-(D3-Pad1): track 0.00 -> 2.38 mm
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