File: Preamp (through-hole-pot)/Preamplifier-with-pots.kicad_pcb (KiCad board)
At the start: 2 copper layers, 100 x 100 mm, 155 parts, among them J1 Conn_01x03_Male, J12 XLR3, J14 Conn_01x03, J15 Conn_01x02, J16 Conn_01x02, J17 Conn_01x02, J2 Conn_01x02_Male, J3 Conn_01x02_Male, J4 Conn_01x03_Male, J5 Conn_01x03_Male, J6 Conn_01x02_Male, J7 Conn_01x03, J8 Conn_01x05_Female, Q1 2N3904, Q2 2N3906, Q3 2N3904, Q4 2N3906, Q5 BC549, SW1 SW_DPST, SW2 SW_SPDT, SW3 GND LIFT, SW4 SW_SPST, SW5 SW_HPFQ, U1 OPA2134, U2 NE5532, U3 NE5532, U4 NE5532, U5 TL072, U6 NE5532, U7 NE5532, U8 NE5532, U9 NE5532

Commit message: More layout
Parts:
- added C31: 0.1uF, Capacitor_SMD:C_0805_2012Metric_Pad1.15x1.40mm_HandSolder, F.Cu at (415.5, 114.8)
- C16, C30, R2, R4, R48: moved to F.Cu
- moved R48 349.7 mm to (420.6, 132.5), turned to 0 degrees
- moved C30 340.7 mm to (411.1, 133.8)
- moved D10 307.1 mm to (384.3, 105.5), turned to 0 degrees
- moved Q5 303.0 mm to (377.5, 120.1)
- moved U5 293.1 mm to (365.9, 113.5), turned to 0 degrees
- moved D12 267.3 mm to (342.5, 117.8)
- moved D13 257.7 mm to (328.4, 108.1)
- moved D7 96.1 mm to (18.0, 59.8), turned to 270 degrees
- moved D2 94.3 mm to (15.2, 59.8), turned to 270 degrees
- moved J5 21.2 mm to (97.5, 97.2)
- moved RV2 21.2 mm to (92.3, 92.2)
- moved J1 11.6 mm to (70.3, 97.0)
- moved RV3 11.1 mm to (28.3, 96.5)
- moved C33 9.28 mm to (38.5, 11.0)
- moved R2 8.75 mm to (5.40, 95.6)
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Connections:
- D13 pad 1: GNDD -> -12V
Routing:
- net +12V: track 129.5 -> 175.6 mm
- net -12V: track 132.5 -> 163.9 mm
- net Net-(R2-Pad1): track 7.47 -> 20.0 mm, vias 0 -> 1
- net Net-(C22-Pad2): track 4.80 -> 0.00 mm
- net Net-(D13-Pad2): track 3.42 -> 0.00 mm
- net Net-(D10-Pad2): track 3.11 -> 0.00 mm
- net Net-(R49-Pad2): track 9.46 -> 6.96 mm
- net Net-(C33-Pad2): track 37.5 -> 35.0 mm
- net Net-(R4-Pad1): track 8.16 -> 10.2 mm, vias 1 -> 0
- net Net-(C4-Pad1): track 7.53 -> 9.36 mm
- net Net-(J2-Pad2): track 4.78 -> 6.27 mm
- net GNDD: track 8.48 -> 7.62 mm
- net GND: vias 11 -> 13
- net (no net): vias 3 -> 0
