File: Preamp (through-hole-pot)/Preamplifier-with-pots.sch (KiCad schematic (older format))
At the start: 155 parts, among them J1 Conn_01x03_Male, J12 XLR3, J14 Conn_01x03, J15 Conn_01x02, J16 Conn_01x02, J17 Conn_01x02, J2 Conn_01x02_Male, J3 Conn_01x02_Male, J4 Conn_01x03_Male, J5 Conn_01x03_Male, J6 Conn_01x02_Male, J7 Conn_01x03, J8 Conn_01x05_Female, Q1 2N3904, Q2 2N3906, Q3 2N3904, Q4 2N3906, Q5 BC549, SW1 SW_DPST, SW2 SW_SPDT, SW3 GND LIFT, SW4 SW_SPST, SW5 SW_HPFQ, U1 OPA2134, U2 NE5532, U3 NE5532, U4 NE5532, U5 TL072, U6 NE5532, U7 NE5532, U8 NE5532, U9 NE5532

Commit message: More layout
Parts:
- added C31: 0.1uF, Capacitor_SMD:C_0805_2012Metric_Pad1.15x1.40mm_HandSolder, symbol Device:C
Connections:
- net -12V: now also D13.1 (K), C31.1
- net GNDD: now also C31.2; no longer D13.1 (K)
Changed lines of the file:
@@
 Wire Wire Line
 	15100 1150 15100 1100
+$Comp
+L power:-12V #PWR0137
+U 1 1 5D762296
+P 15100 1850
+F 0 "#PWR0137" H 15100 1950 50  0001 C CNN
+F 1 "-12V" H 15115 2023 50  0000 C CNN
+F 2 "" H 15100 1850 50  0001 C CNN
+F 3 "" H 15100 1850 50  0001 C CNN
+	1    15100 1850
+	-1   0    0    1
+$EndComp
 Wire Wire Line
 	15100 1850 15100 1800
@@
 $EndComp
 $Comp
+L power:-12V #PWR0142
+U 1 1 5D7B4AE2
+P 15100 3100
+F 0 "#PWR0142" H 15100 3200 50  0001 C CNN
+F 1 "-12V" H 15115 3273 50  0000 C CNN
+F 2 "" H 15100 3100 50  0001 C CNN
+F 3 "" H 15100 3100 50  0001 C CNN
+	1    15100 3100
+	-1   0    0    1
+$EndComp
+$Comp
+L Device:C C31
+U 1 1 5D7B4AEE
+P 15100 2950
+F 0 "C31" H 14985 2904 50  0000 R CNN
+F 1 "0.1uF" H 14985 2995 50  0000 R CNN
+F 2 "Capacitor_SMD:C_0805_2012Metric_Pad1.15x1.40mm_HandSolder" H 15138 2800 50  0001 C CNN
+F 3 "~" H 15100 2950 50  0001 C CNN
+	1    15100 2950
+	-1   0    0    1
+$EndComp
+$Comp
 L Device:C C30
 U 1 1 5D7B4AF4
@@
 L power:GNDD #PWR0210
 U 1 1 5E337C4E
-P 15100 2800
-F 0 "#PWR0210" H 15100 2550 50  0001 C CNN
-F 1 "GNDD" H 15104 2645 50  0000 C CNN
-F 2 "" H 15100 2800 50  0001 C CNN
-F 3 "" H 15100 2800 50  0001 C CNN
-	1    15100 2800
+P 14850 2800
+F 0 "#PWR0210" H 14850 2550 50  0001 C CNN
+F 1 "GNDD" H 14854 2645 50  0000 C CNN
+F 2 "" H 14850 2800 50  0001 C CNN
+F 3 "" H 14850 2800 50  0001 C CNN
+	1    14850 2800
 	1    0    0    -1
 $EndComp
@@
 Wire Wire Line
 	15100 2750 15100 2800
+Wire Wire Line
+	15100 2800 14850 2800
+Connection ~ 15100 2800
 $Comp
 L Connector:Conn_01x02_Male J2
@@
 	1    0    0    -1
 $EndComp
-$Comp
-L power:GNDD #PWR?
-U 1 1 5E43DBBD
-P 15100 1850
-F 0 "#PWR?" H 15100 1600 50  0001 C CNN
-F 1 "GNDD" H 15104 1695 50  0000 C CNN
-F 2 "" H 15100 1850 50  0001 C CNN
-F 3 "" H 15100 1850 50  0001 C CNN
-	1    15100 1850
-	1    0    0    -1
-$EndComp
